Commit message: removed prints, updated todo

File: testrobot.urdf (robot description, URDF)
Before this commit: robot testrobot, 2 links, 0 joints
Links:
- removed link base_link
- removed link box_one 
- added link base_box; visual box size=1 1 1
- added link base_sphere; visual sphere radius=0.5
Joints:
- added joint box_to_sphere: type fixed, parent base_box, child base_sphere
