Commit message: data.yaml um link funktion erweitert

File: preview_robot.urdf (robot description, URDF)
Before this commit: robot testrobot, 2 links, 1 joints
Links:
- removed link base_box
- removed link base_sphere
- added link box_one; visual box size=1 1 1
- added link sphere_one; visual sphere radius=0.5
Joints:
- removed joint box_to_sphere
