Commit message: Refactor

File: World Generator/maze.urdf (robot description, URDF)
Before this commit: robot maze, 145 links, 144 joints
Links:
- link link_0: geometry collision box size=0.35 0.05 0.5; visual box size=0.35 0.05 0.5
- link link_1: geometry collision box size=0.05 0.35 0.5; visual box size=0.05 0.35 0.5
- link link_10: geometry collision box size=0.35 0.05 0.5; visual box size=0.35 0.05 0.5
- link link_100: geometry collision box size=0.35 0.05 0.5; visual box size=0.35 0.05 0.5
- link link_101: geometry collision box size=0.05 0.35 0.5; visual box size=0.05 0.35 0.5
- link link_102: geometry collision box size=0.35 0.05 0.5; visual box size=0.35 0.05 0.5
- link link_103: geometry collision box size=0.05 0.35 0.5; visual box size=0.05 0.35 0.5
- link link_104: geometry collision box size=0.05 0.35 0.5; visual box size=0.05 0.35 0.5
- link link_105: geometry collision box size=0.05 0.35 0.5; visual box size=0.05 0.35 0.5
- link link_106: geometry collision box size=0.05 0.35 0.5; visual box size=0.05 0.35 0.5
- link link_107: geometry collision box size=0.05 0.35 0.5; visual box size=0.05 0.35 0.5
- link link_108: geometry collision box size=0.05 0.35 0.5; visual box size=0.05 0.35 0.5
- link link_109: geometry collision box size=0.05 0.35 0.5; visual box size=0.05 0.35 0.5
- link link_11: geometry collision box size=0.05 0.35 0.5; visual box size=0.05 0.35 0.5
- link link_110: geometry collision box size=0.35 0.05 0.5; visual box size=0.35 0.05 0.5
- link link_111: geometry collision box size=0.35 0.05 0.5; visual box size=0.35 0.05 0.5
- link link_112: geometry collision box size=0.35 0.05 0.5; visual box size=0.35 0.05 0.5
- link link_113: geometry collision box size=0.35 0.05 0.5; visual box size=0.35 0.05 0.5
- link link_114: geometry collision box size=0.35 0.05 0.5; visual box size=0.35 0.05 0.5
- link link_115: geometry collision box size=0.35 0.05 0.5; visual box size=0.35 0.05 0.5
- link link_116: geometry collision box size=0.05 0.35 0.5; visual box size=0.05 0.35 0.5
- link link_117: geometry collision box size=0.05 0.35 0.5; visual box size=0.05 0.35 0.5
- link link_118: geometry collision box size=0.05 0.35 0.5; visual box size=0.05 0.35 0.5
- link link_119: geometry collision box size=0.05 0.35 0.5; visual box size=0.05 0.35 0.5
- link link_12: geometry collision box size=0.35 0.05 0.5; visual box size=0.35 0.05 0.5
- link link_120: geometry collision box size=0.05 0.35 0.5; visual box size=0.05 0.35 0.5
- link link_121: geometry collision box size=0.05 0.6 0.25; visual box size=0.05 0.6 0.25
- link link_122: geometry collision box size=0.05 0.35 0.5; visual box size=0.05 0.35 0.5
- link link_123: geometry collision box size=0.05 0.35 0.5; visual box size=0.05 0.35 0.5
- link link_124: geometry collision box size=0.05 0.35 0.5; visual box size=0.05 0.35 0.5
- link link_125: geometry collision box size=0.05 0.35 0.5; visual box size=0.05 0.35 0.5
- link link_126: geometry collision box size=0.35 0.05 0.5; visual box size=0.35 0.05 0.5
- link link_127: geometry collision box size=0.35 0.05 0.5; visual box size=0.35 0.05 0.5
- link link_128: geometry collision box size=0.35 0.05 0.5; visual box size=0.35 0.05 0.5
- link link_129: geometry collision box size=0.35 0.05 0.5; visual box size=0.35 0.05 0.5
- link link_13: geometry collision box size=0.35 0.05 0.5; visual box size=0.35 0.05 0.5
- link link_130: geometry collision box size=0.35 0.05 0.5; visual box size=0.35 0.05 0.5
- link link_131: geometry collision box size=0.35 0.05 0.5; visual box size=0.35 0.05 0.5
- link link_132: geometry collision box size=0.35 0.05 0.5; visual box size=0.35 0.05 0.5
- link link_133: geometry collision box size=0.35 0.05 0.5; visual box size=0.35 0.05 0.5
- link link_134: geometry collision box size=0.35 0.05 0.5; visual box size=0.35 0.05 0.5
- link link_135: geometry collision box size=0.35 0.05 0.5; visual box size=0.35 0.05 0.5
- link link_136: geometry collision box size=0.35 0.05 0.5; visual box size=0.35 0.05 0.5
- link link_137: geometry collision box size=0.35 0.05 0.5; visual box size=0.35 0.05 0.5
- link link_138: geometry collision box size=0.35 0.05 0.5; visual box size=0.35 0.05 0.5
- link link_139: geometry collision box size=0.35 0.05 0.5; visual box size=0.35 0.05 0.5
- link link_14: geometry collision box size=0.05 0.35 0.5; visual box size=0.05 0.35 0.5
- link link_140: geometry collision box size=0.35 0.05 0.5; visual box size=0.35 0.05 0.5
- link link_141: geometry collision box size=0.35 0.05 0.5; visual box size=0.35 0.05 0.5
- link link_142: geometry collision box size=0.35 0.05 0.5; visual box size=0.35 0.05 0.5
- link link_143: geometry collision box size=0.35 0.05 0.5; visual box size=0.35 0.05 0.5
- link link_15: geometry collision box size=0.35 0.05 0.5; visual box size=0.35 0.05 0.5
- link link_16: geometry collision box size=0.35 0.05 0.5; visual box size=0.35 0.05 0.5
- link link_17: geometry collision box size=0.35 0.05 0.5; visual box size=0.35 0.05 0.5
- link link_18: geometry collision box size=0.35 0.05 0.5; visual box size=0.35 0.05 0.5
- link link_19: geometry collision box size=0.35 0.05 0.5; visual box size=0.35 0.05 0.5
- link link_2: geometry collision box size=0.35 0.05 0.5; visual box size=0.35 0.05 0.5
- link link_20: geometry collision box size=0.35 0.05 0.5; visual box size=0.35 0.05 0.5
- link link_21: geometry collision box size=0.35 0.05 0.5; visual box size=0.35 0.05 0.5
- link link_22: geometry collision box size=0.05 0.35 0.5; visual box size=0.05 0.35 0.5
- link link_23: geometry collision box size=0.05 0.35 0.5; visual box size=0.05 0.35 0.5
- link link_24: geometry collision box size=0.05 0.35 0.5; visual box size=0.05 0.35 0.5
- link link_25: geometry collision box size=0.05 0.35 0.5; visual box size=0.05 0.35 0.5
- link link_26: geometry collision box size=0.05 0.35 0.5; visual box size=0.05 0.35 0.5
- link link_27: geometry collision box size=0.05 0.35 0.5; visual box size=0.05 0.35 0.5
- link link_28: geometry collision box size=0.05 0.35 0.5; visual box size=0.05 0.35 0.5
- link link_29: geometry collision box size=0.05 0.35 0.5; visual box size=0.05 0.35 0.5
- link link_3: geometry collision box size=0.35 0.05 0.5; visual box size=0.35 0.05 0.5
- link link_30: geometry collision box size=0.6 0.05 0.25; visual box size=0.6 0.05 0.25
- link link_31: geometry collision box size=0.05 0.35 0.5; visual box size=0.05 0.35 0.5
- link link_32: geometry collision box size=0.05 0.35 0.5; visual box size=0.05 0.35 0.5
- link link_33: geometry collision box size=0.05 0.35 0.5; visual box size=0.05 0.35 0.5
- link link_34: geometry collision box size=0.05 0.35 0.5; visual box size=0.05 0.35 0.5
- link link_35: geometry collision box size=0.6 0.05 0.25; visual box size=0.6 0.05 0.25
- link link_36: geometry collision box size=0.05 0.35 0.5; visual box size=0.05 0.35 0.5
- link link_37: geometry collision box size=0.05 0.35 0.5; visual box size=0.05 0.35 0.5
- link link_38: geometry collision box size=0.05 0.35 0.5; visual box size=0.05 0.35 0.5
- link link_39: geometry collision box size=0.05 0.35 0.5; visual box size=0.05 0.35 0.5
- link link_4: geometry collision box size=0.35 0.05 0.5; visual box size=0.35 0.05 0.5
- link link_40: geometry collision box size=0.6 0.05 0.25; visual box size=0.6 0.05 0.25
- link link_41: geometry collision box size=0.05 0.35 0.5; visual box size=0.05 0.35 0.5
- link link_42: geometry collision box size=0.05 0.35 0.5; visual box size=0.05 0.35 0.5
- link link_43: geometry collision box size=0.05 0.35 0.5; visual box size=0.05 0.35 0.5
- link link_44: geometry collision box size=0.05 0.35 0.5; visual box size=0.05 0.35 0.5
- link link_45: geometry collision box size=0.05 0.35 0.5; visual box size=0.05 0.35 0.5
- link link_46: geometry collision box size=0.05 0.35 0.5; visual box size=0.05 0.35 0.5
- link link_47: geometry collision box size=0.05 0.35 0.5; visual box size=0.05 0.35 0.5
- link link_48: geometry collision box size=0.05 0.35 0.5; visual box size=0.05 0.35 0.5
- link link_49: geometry collision box size=0.05 0.35 0.5; visual box size=0.05 0.35 0.5
- link link_5: geometry collision box size=0.35 0.05 0.5; visual box size=0.35 0.05 0.5
- link link_50: geometry collision box size=0.05 0.35 0.5; visual box size=0.05 0.35 0.5
- link link_51: geometry collision box size=0.05 0.35 0.5; visual box size=0.05 0.35 0.5
- link link_52: geometry collision box size=0.35 0.05 0.5; visual box size=0.35 0.05 0.5
- link link_53: geometry collision box size=0.35 0.05 0.5; visual box size=0.35 0.05 0.5
- link link_54: geometry collision box size=0.05 0.35 0.5; visual box size=0.05 0.35 0.5
- link link_55: geometry collision box size=0.35 0.05 0.5; visual box size=0.35 0.05 0.5
- link link_56: geometry collision box size=0.35 0.05 0.5; visual box size=0.35 0.05 0.5
- link link_57: geometry collision box size=0.05 0.35 0.5; visual box size=0.05 0.35 0.5
- link link_58: geometry collision box size=0.05 0.35 0.5; visual box size=0.05 0.35 0.5
- link link_59: geometry collision box size=0.05 0.35 0.5; visual box size=0.05 0.35 0.5
- link link_6: geometry collision box size=0.05 0.35 0.5; visual box size=0.05 0.35 0.5
- link link_60: geometry collision box size=0.05 0.35 0.5; visual box size=0.05 0.35 0.5
- link link_61: geometry collision box size=0.05 0.35 0.5; visual box size=0.05 0.35 0.5
- link link_62: geometry collision box size=0.05 0.35 0.5; visual box size=0.05 0.35 0.5
- link link_63: geometry collision box size=0.05 0.35 0.5; visual box size=0.05 0.35 0.5
- link link_64: geometry collision box size=0.05 0.35 0.5; visual box size=0.05 0.35 0.5
- link link_65: geometry collision box size=0.05 0.35 0.5; visual box size=0.05 0.35 0.5
- link link_66: geometry collision box size=0.35 0.05 0.5; visual box size=0.35 0.05 0.5
- link link_67: geometry collision box size=0.05 0.35 0.5; visual box size=0.05 0.35 0.5
- link link_68: geometry collision box size=0.35 0.05 0.5; visual box size=0.35 0.05 0.5
- link link_69: geometry collision box size=0.35 0.05 0.5; visual box size=0.35 0.05 0.5
- link link_7: geometry collision box size=0.35 0.05 0.5; visual box size=0.35 0.05 0.5
- link link_70: geometry collision box size=0.35 0.05 0.5; visual box size=0.35 0.05 0.5
- link link_71: geometry collision box size=0.35 0.05 0.5; visual box size=0.35 0.05 0.5
- link link_72: geometry collision box size=0.05 0.35 0.5; visual box size=0.05 0.35 0.5
- link link_73: geometry collision box size=0.35 0.05 0.5; visual box size=0.35 0.05 0.5
- link link_74: geometry collision box size=0.35 0.05 0.5; visual box size=0.35 0.05 0.5
- link link_75: geometry collision box size=0.35 0.05 0.5; visual box size=0.35 0.05 0.5
- link link_76: geometry collision box size=0.35 0.05 0.5; visual box size=0.35 0.05 0.5
- link link_77: geometry collision box size=0.35 0.05 0.5; visual box size=0.35 0.05 0.5
- link link_78: geometry collision box size=0.35 0.05 0.5; visual box size=0.35 0.05 0.5
- link link_79: geometry collision box size=0.05 0.35 0.5; visual box size=0.05 0.35 0.5
- link link_8: geometry collision box size=0.35 0.05 0.5; visual box size=0.35 0.05 0.5
- link link_80: geometry collision box size=0.35 0.05 0.5; visual box size=0.35 0.05 0.5
- link link_81: geometry collision box size=0.6 0.05 0.25; visual box size=0.6 0.05 0.25
- link link_82: geometry collision box size=0.05 0.35 0.5; visual box size=0.05 0.35 0.5
- link link_83: geometry collision box size=0.05 0.35 0.5; visual box size=0.05 0.35 0.5
- link link_84: geometry collision box size=0.05 0.35 0.5; visual box size=0.05 0.35 0.5
- link link_85: geometry collision box size=0.05 0.35 0.5; visual box size=0.05 0.35 0.5
- link link_86: geometry collision box size=0.05 0.35 0.5; visual box size=0.05 0.35 0.5
- link link_87: geometry collision box size=0.05 0.35 0.5; visual box size=0.05 0.35 0.5
- link link_88: geometry collision box size=0.05 0.35 0.5; visual box size=0.05 0.35 0.5
- link link_89: geometry collision box size=0.05 0.35 0.5; visual box size=0.05 0.35 0.5
- link link_9: geometry collision box size=0.35 0.05 0.5; visual box size=0.35 0.05 0.5
- link link_90: geometry collision box size=0.05 0.35 0.5; visual box size=0.05 0.35 0.5
- link link_91: geometry collision box size=0.05 0.35 0.5; visual box size=0.05 0.35 0.5
- link link_92: geometry collision box size=0.05 0.35 0.5; visual box size=0.05 0.35 0.5
- link link_93: geometry collision box size=0.35 0.05 0.5; visual box size=0.35 0.05 0.5
- link link_94: geometry collision box size=0.35 0.05 0.5; visual box size=0.35 0.05 0.5
- link link_95: geometry collision box size=0.35 0.05 0.5; visual box size=0.35 0.05 0.5
- link link_96: geometry collision box size=0.35 0.05 0.5; visual box size=0.35 0.05 0.5
- link link_97: geometry collision box size=0.6 0.05 0.25; visual box size=0.6 0.05 0.25
- link link_98: geometry collision box size=0.35 0.05 0.5; visual box size=0.35 0.05 0.5
- link link_99: geometry collision box size=0.35 0.05 0.5; visual box size=0.35 0.05 0.5

Commit message: more refactoring

File: World Generator/maze.urdf (robot description, URDF)
Before this commit: robot maze, 145 links, 144 joints
Links:
- link link_100: geometry collision box size=0.05 0.35 0.5; visual box size=0.05 0.35 0.5
- link link_102: geometry collision box size=0.05 0.6 0.25; visual box size=0.05 0.6 0.25
- link link_103: geometry collision box size=0.05 0.6 0.25; visual box size=0.05 0.6 0.25
- link link_11: geometry collision box size=0.35 0.05 0.5; visual box size=0.35 0.05 0.5
- link link_116: geometry collision box size=0.35 0.05 0.5; visual box size=0.35 0.05 0.5
- link link_117: geometry collision box size=0.35 0.05 0.5; visual box size=0.35 0.05 0.5
- link link_121: geometry collision box size=0.05 0.35 0.5; visual box size=0.05 0.35 0.5
- link link_122: geometry collision box size=0.05 0.6 0.25; visual box size=0.05 0.6 0.25
- link link_14: geometry collision box size=0.35 0.05 0.5; visual box size=0.35 0.05 0.5
- link link_20: geometry collision box size=0.05 0.35 0.5; visual box size=0.05 0.35 0.5
- link link_21: geometry collision box size=0.05 0.35 0.5; visual box size=0.05 0.35 0.5
- link link_25: geometry collision box size=0.35 0.05 0.5; visual box size=0.35 0.05 0.5
- link link_26: geometry collision box size=0.35 0.05 0.5; visual box size=0.35 0.05 0.5
- link link_29: geometry collision box size=0.35 0.05 0.5; visual box size=0.35 0.05 0.5
- link link_30: geometry collision box size=0.35 0.05 0.5; visual box size=0.35 0.05 0.5
- link link_31: geometry collision box size=0.35 0.05 0.5; visual box size=0.35 0.05 0.5
- link link_32: geometry collision box size=0.35 0.05 0.5; visual box size=0.35 0.05 0.5
- link link_33: geometry collision box size=0.35 0.05 0.5; visual box size=0.35 0.05 0.5
- link link_34: geometry collision box size=0.35 0.05 0.5; visual box size=0.35 0.05 0.5
- link link_35: geometry collision box size=0.35 0.05 0.5; visual box size=0.35 0.05 0.5
- link link_36: geometry collision box size=0.35 0.05 0.5; visual box size=0.35 0.05 0.5
- link link_40: geometry collision box size=0.05 0.35 0.5; visual box size=0.05 0.35 0.5
- link link_44: geometry collision box size=0.35 0.05 0.5; visual box size=0.35 0.05 0.5
- link link_46: geometry collision box size=0.35 0.05 0.5; visual box size=0.35 0.05 0.5
- link link_47: geometry collision box size=0.35 0.05 0.5; visual box size=0.35 0.05 0.5
- link link_48: geometry collision box size=0.35 0.05 0.5; visual box size=0.35 0.05 0.5
- link link_49: geometry collision box size=0.35 0.05 0.5; visual box size=0.35 0.05 0.5
- link link_50: geometry collision box size=0.35 0.05 0.5; visual box size=0.35 0.05 0.5
- link link_51: geometry collision box size=0.35 0.05 0.5; visual box size=0.35 0.05 0.5
- link link_52: geometry collision box size=0.05 0.35 0.5; visual box size=0.05 0.35 0.5
- link link_54: geometry collision box size=0.35 0.05 0.5; visual box size=0.35 0.05 0.5
- link link_57: geometry collision box size=0.35 0.05 0.5; visual box size=0.35 0.05 0.5
- link link_58: geometry collision box size=0.6 0.05 0.25; visual box size=0.6 0.05 0.25
- link link_6: geometry collision box size=0.35 0.05 0.5; visual box size=0.35 0.05 0.5
- link link_66: geometry collision box size=0.05 0.35 0.5; visual box size=0.05 0.35 0.5
- link link_67: geometry collision box size=0.35 0.05 0.5; visual box size=0.35 0.05 0.5
- link link_70: geometry collision box size=0.05 0.35 0.5; visual box size=0.05 0.35 0.5
- link link_72: geometry collision box size=0.35 0.05 0.5; visual box size=0.35 0.05 0.5
- link link_73: geometry collision box size=0.05 0.35 0.5; visual box size=0.05 0.35 0.5
- link link_77: geometry collision box size=0.05 0.35 0.5; visual box size=0.05 0.35 0.5
- link link_78: geometry collision box size=0.05 0.35 0.5; visual box size=0.05 0.35 0.5
- link link_8: geometry collision box size=0.05 0.35 0.5; visual box size=0.05 0.35 0.5
- link link_80: geometry collision box size=0.05 0.35 0.5; visual box size=0.05 0.35 0.5
- link link_81: geometry collision box size=0.05 0.35 0.5; visual box size=0.05 0.35 0.5
- link link_85: geometry collision box size=0.35 0.05 0.5; visual box size=0.35 0.05 0.5
- link link_87: geometry collision box size=0.35 0.05 0.5; visual box size=0.35 0.05 0.5
- link link_88: geometry collision box size=0.35 0.05 0.5; visual box size=0.35 0.05 0.5
- link link_89: geometry collision box size=0.35 0.05 0.5; visual box size=0.35 0.05 0.5
- link link_90: geometry collision box size=0.35 0.05 0.5; visual box size=0.35 0.05 0.5
- link link_91: geometry collision box size=0.35 0.05 0.5; visual box size=0.35 0.05 0.5
- link link_94: geometry collision box size=0.05 0.35 0.5; visual box size=0.05 0.35 0.5
- link link_96: geometry collision box size=0.05 0.35 0.5; visual box size=0.05 0.35 0.5
- link link_97: geometry collision box size=0.35 0.05 0.5; visual box size=0.35 0.05 0.5
- link link_98: geometry collision box size=0.05 0.35 0.5; visual box size=0.05 0.35 0.5

Commit message: humanoid

File: World Generator/maze.urdf (robot description, URDF)
Before this commit: robot maze, 145 links, 144 joints
Links:
- added link link_144; collision box size=0.35 0.05 0.5; visual box size=0.35 0.05 0.5
- added link link_145; collision box size=0.35 0.05 0.5; visual box size=0.35 0.05 0.5
- link link_10: geometry collision box size=0.05 0.35 0.5; visual box size=0.05 0.35 0.5
- link link_100: geometry collision box size=0.35 0.05 0.5; visual box size=0.35 0.05 0.5
- link link_102: geometry collision box size=0.05 0.35 0.5; visual box size=0.05 0.35 0.5
- link link_103: geometry collision box size=0.05 0.35 0.5; visual box size=0.05 0.35 0.5
- link link_105: geometry collision box size=0.05 0.6 0.25; visual box size=0.05 0.6 0.25
- link link_109: geometry collision box size=0.35 0.05 0.5; visual box size=0.35 0.05 0.5
- link link_113: geometry collision box size=0.05 0.35 0.5; visual box size=0.05 0.35 0.5
- link link_118: geometry collision box size=0.35 0.05 0.5; visual box size=0.35 0.05 0.5
- link link_119: geometry collision box size=0.35 0.05 0.5; visual box size=0.35 0.05 0.5
- link link_120: geometry collision box size=0.35 0.05 0.5; visual box size=0.35 0.05 0.5
- link link_121: geometry collision box size=0.35 0.05 0.5; visual box size=0.35 0.05 0.5
- link link_122: geometry collision box size=0.05 0.35 0.5; visual box size=0.05 0.35 0.5
- link link_124: geometry collision box size=0.05 0.6 0.25; visual box size=0.05 0.6 0.25
- link link_126: geometry collision box size=0.05 0.6 0.25; visual box size=0.05 0.6 0.25
- link link_127: geometry collision box size=0.05 0.35 0.5; visual box size=0.05 0.35 0.5
- link link_23: geometry collision box size=0.05 0.6 0.25; visual box size=0.05 0.6 0.25
- link link_25: geometry collision box size=0.05 0.35 0.5; visual box size=0.05 0.35 0.5
- link link_28: geometry collision box size=0.35 0.05 0.5; visual box size=0.35 0.05 0.5
- link link_31: geometry collision box size=0.05 0.35 0.5; visual box size=0.05 0.35 0.5
- link link_38: geometry collision box size=0.35 0.05 0.5; visual box size=0.35 0.05 0.5
- link link_43: geometry collision box size=0.05 0.6 0.25; visual box size=0.05 0.6 0.25
- link link_44: geometry collision box size=0.05 0.35 0.5; visual box size=0.05 0.35 0.5
- link link_46: geometry collision box size=0.05 0.35 0.5; visual box size=0.05 0.35 0.5
- link link_47: geometry collision box size=0.05 0.35 0.5; visual box size=0.05 0.35 0.5
- link link_48: geometry collision box size=0.6 0.05 0.25; visual box size=0.6 0.05 0.25
- link link_50: geometry collision box size=0.05 0.35 0.5; visual box size=0.05 0.35 0.5
- link link_52: geometry collision box size=0.35 0.05 0.5; visual box size=0.35 0.05 0.5
- link link_57: geometry collision box size=0.05 0.35 0.5; visual box size=0.05 0.35 0.5
- link link_58: geometry collision box size=0.35 0.05 0.5; visual box size=0.35 0.05 0.5
- link link_59: geometry collision box size=0.35 0.05 0.5; visual box size=0.35 0.05 0.5
- link link_60: geometry collision box size=0.35 0.05 0.5; visual box size=0.35 0.05 0.5
- link link_67: geometry collision box size=0.05 0.35 0.5; visual box size=0.05 0.35 0.5
- link link_71: geometry collision box size=0.05 0.35 0.5; visual box size=0.05 0.35 0.5
- link link_73: geometry collision box size=0.35 0.05 0.5; visual box size=0.35 0.05 0.5
- link link_78: geometry collision box size=0.35 0.05 0.5; visual box size=0.35 0.05 0.5
- link link_8: geometry collision box size=0.35 0.05 0.5; visual box size=0.35 0.05 0.5
- link link_85: geometry collision box size=0.05 0.35 0.5; visual box size=0.05 0.35 0.5
- link link_88: geometry collision box size=0.05 0.35 0.5; visual box size=0.05 0.35 0.5
- link link_90: geometry collision box size=0.05 0.35 0.5; visual box size=0.05 0.35 0.5
- link link_92: geometry collision box size=0.35 0.05 0.5; visual box size=0.35 0.05 0.5
- link link_98: geometry collision box size=0.35 0.05 0.5; visual box size=0.35 0.05 0.5
Joints:
- added joint joint_144: type fixed, parent base_link, child link_144, origin xyz=0 0 0 rpy=0 0 0
- added joint joint_145: type fixed, parent base_link, child link_145, origin xyz=0 0 0 rpy=0 0 0
