Commit message: bugfix

File: urdfs/generated/shelf.urdf (robot description, URDF)
Before this commit: robot maze, 263 links, 262 joints
Links:
- removed link link_123
- removed link link_124
- removed link link_125
- removed link link_126
- removed link link_127
- removed link link_128
- removed link link_129
- removed link link_130
- removed link link_131
- removed link link_132
- removed link link_133
- removed link link_134
- removed link link_135
- removed link link_136
- removed link link_137
- removed link link_138
- removed link link_139
- removed link link_140
- removed link link_141
- removed link link_142
- removed link link_143
- removed link link_144
- removed link link_145
- removed link link_146
- removed link link_147
- removed link link_148
- removed link link_149
- removed link link_150
- removed link link_151
- removed link link_152
- removed link link_153
- removed link link_154
- removed link link_155
- removed link link_156
- removed link link_157
- removed link link_158
- removed link link_159
- removed link link_160
- removed link link_161
- removed link link_162
- removed link link_163
- removed link link_164
- removed link link_165
- removed link link_166
- removed link link_167
- removed link link_168
- removed link link_169
- removed link link_170
- removed link link_171
- removed link link_172
- removed link link_173
- removed link link_174
- removed link link_175
- removed link link_176
- removed link link_177
- removed link link_178
- removed link link_179
- removed link link_180
- removed link link_181
- removed link link_182
- removed link link_183
- removed link link_184
- removed link link_185
- removed link link_186
- removed link link_187
- removed link link_188
- removed link link_189
- removed link link_190
- removed link link_191
- removed link link_192
- removed link link_193
- removed link link_194
- removed link link_195
- removed link link_196
- removed link link_197
- removed link link_198
- removed link link_199
- removed link link_200
- removed link link_201
- removed link link_202
- removed link link_203
- removed link link_204
- removed link link_205
- removed link link_206
- removed link link_207
- removed link link_208
- removed link link_209
- removed link link_210
- removed link link_211
- removed link link_212
- removed link link_213
- removed link link_214
- removed link link_215
- removed link link_216
- removed link link_217
- removed link link_218
- removed link link_219
- removed link link_220
- removed link link_221
- removed link link_222
- removed link link_223
- removed link link_224
- removed link link_225
- removed link link_226
- removed link link_227
- removed link link_228
- removed link link_229
- removed link link_230
- removed link link_231
- removed link link_232
- removed link link_233
- removed link link_234
- removed link link_235
- removed link link_236
- removed link link_237
- removed link link_238
- removed link link_239
- removed link link_240
- removed link link_241
- removed link link_242
- removed link link_243
- removed link link_244
- removed link link_245
- removed link link_246
- removed link link_247
- removed link link_248
- removed link link_249
- removed link link_250
- removed link link_251
- removed link link_252
- removed link link_253
- removed link link_254
- removed link link_255
- removed link link_256
- removed link link_257
- removed link link_258
- removed link link_259
- removed link link_260
- removed link link_261
- link link_0: geometry collision box size=0.21000000000000002 0.01 0.5; visual box size=0.21000000000000002 0.01 0.5
- link link_1: geometry collision box size=0.01 0.21000000000000002 0.5; visual box size=0.01 0.21000000000000002 0.5
- link link_10: geometry collision box size=0.21000000000000002 0.01 0.5; visual box size=0.21000000000000002 0.01 0.5
- link link_100: geometry collision box size=0.01 0.21000000000000002 0.5; visual box size=0.01 0.21000000000000002 0.5
- link link_101: geometry collision box size=0.21000000000000002 0.01 0.5; visual box size=0.21000000000000002 0.01 0.5
- link link_102: geometry collision box size=0.01 0.21000000000000002 0.5; visual box size=0.01 0.21000000000000002 0.5
- link link_103: geometry collision box size=0.01 0.21000000000000002 0.5; visual box size=0.01 0.21000000000000002 0.5
- link link_104: geometry collision box size=0.21000000000000002 0.01 0.5; visual box size=0.21000000000000002 0.01 0.5
- link link_105: geometry collision box size=0.01 0.21000000000000002 0.5; visual box size=0.01 0.21000000000000002 0.5
- link link_106: geometry collision box size=0.21000000000000002 0.01 0.5; visual box size=0.21000000000000002 0.01 0.5
- link link_107: geometry collision box size=0.21000000000000002 0.01 0.5; visual box size=0.21000000000000002 0.01 0.5
- link link_108: geometry collision box size=0.01 0.21000000000000002 0.5; visual box size=0.01 0.21000000000000002 0.5
- link link_109: geometry collision box size=0.21000000000000002 0.01 0.5; visual box size=0.21000000000000002 0.01 0.5
- link link_11: geometry collision box size=0.01 0.21000000000000002 0.5; visual box size=0.01 0.21000000000000002 0.5
- link link_110: geometry collision box size=0.21000000000000002 0.01 0.5; visual box size=0.21000000000000002 0.01 0.5
- link link_111: geometry collision box size=0.01 0.21000000000000002 0.5; visual box size=0.01 0.21000000000000002 0.5
- link link_112: geometry collision box size=0.21000000000000002 0.01 0.5; visual box size=0.21000000000000002 0.01 0.5
- link link_113: geometry collision box size=0.21000000000000002 0.01 0.5; visual box size=0.21000000000000002 0.01 0.5
- link link_114: geometry collision box size=0.01 0.21000000000000002 0.5; visual box size=0.01 0.21000000000000002 0.5
- link link_115: geometry collision box size=0.21000000000000002 0.01 0.5; visual box size=0.21000000000000002 0.01 0.5
- link link_116: geometry collision box size=0.21000000000000002 0.01 0.5; visual box size=0.21000000000000002 0.01 0.5
- link link_117: geometry collision box size=0.01 0.21000000000000002 0.5; visual box size=0.01 0.21000000000000002 0.5
- link link_118: geometry collision box size=0.21000000000000002 0.01 0.5; visual box size=0.21000000000000002 0.01 0.5
- link link_119: geometry collision box size=0.21000000000000002 0.01 0.5; visual box size=0.21000000000000002 0.01 0.5
- link link_12: geometry collision box size=0.01 0.21000000000000002 0.5; visual box size=0.01 0.21000000000000002 0.5
- link link_120: geometry collision box size=0.01 0.21000000000000002 0.5; visual box size=0.01 0.21000000000000002 0.5
- link link_121: geometry collision box size=0.01 0.21000000000000002 0.5; visual box size=0.01 0.21000000000000002 0.5
- link link_122: geometry collision box size=0.21000000000000002 0.01 0.5; visual box size=0.21000000000000002 0.01 0.5
- link link_13: geometry collision box size=0.21000000000000002 0.01 0.5; visual box size=0.21000000000000002 0.01 0.5
- link link_14: geometry collision box size=0.01 0.21000000000000002 0.5; visual box size=0.01 0.21000000000000002 0.5
- link link_15: geometry collision box size=0.21000000000000002 0.01 0.5; visual box size=0.21000000000000002 0.01 0.5
- link link_16: geometry collision box size=0.01 0.21000000000000002 0.5; visual box size=0.01 0.21000000000000002 0.5
- link link_17: geometry collision box size=0.21000000000000002 0.01 0.5; visual box size=0.21000000000000002 0.01 0.5
- link link_18: geometry collision box size=0.01 0.21000000000000002 0.5; visual box size=0.01 0.21000000000000002 0.5
- link link_19: geometry collision box size=0.21000000000000002 0.01 0.5; visual box size=0.21000000000000002 0.01 0.5
- link link_2: geometry collision box size=0.21000000000000002 0.01 0.5; visual box size=0.21000000000000002 0.01 0.5
- link link_20: geometry collision box size=0.01 0.21000000000000002 0.5; visual box size=0.01 0.21000000000000002 0.5
- link link_21: geometry collision box size=0.21000000000000002 0.01 0.5; visual box size=0.21000000000000002 0.01 0.5
- link link_22: geometry collision box size=0.01 0.21000000000000002 0.5; visual box size=0.01 0.21000000000000002 0.5
- link link_23: geometry collision box size=0.21000000000000002 0.01 0.5; visual box size=0.21000000000000002 0.01 0.5
- link link_24: geometry collision box size=0.01 0.21000000000000002 0.5; visual box size=0.01 0.21000000000000002 0.5
- link link_25: geometry collision box size=0.01 0.21000000000000002 0.5; visual box size=0.01 0.21000000000000002 0.5
- link link_26: geometry collision box size=0.21000000000000002 0.01 0.5; visual box size=0.21000000000000002 0.01 0.5
- link link_27: geometry collision box size=0.01 0.21000000000000002 0.5; visual box size=0.01 0.21000000000000002 0.5
- link link_28: geometry collision box size=0.21000000000000002 0.01 0.5; visual box size=0.21000000000000002 0.01 0.5
- link link_29: geometry collision box size=0.01 0.21000000000000002 0.5; visual box size=0.01 0.21000000000000002 0.5
- link link_3: geometry collision box size=0.01 0.21000000000000002 0.5; visual box size=0.01 0.21000000000000002 0.5
- link link_30: geometry collision box size=0.21000000000000002 0.01 0.5; visual box size=0.21000000000000002 0.01 0.5
- link link_31: geometry collision box size=0.01 0.21000000000000002 0.5; visual box size=0.01 0.21000000000000002 0.5
- link link_32: geometry collision box size=0.21000000000000002 0.01 0.5; visual box size=0.21000000000000002 0.01 0.5
- link link_33: geometry collision box size=0.01 0.21000000000000002 0.5; visual box size=0.01 0.21000000000000002 0.5
- link link_34: geometry collision box size=0.21000000000000002 0.01 0.5; visual box size=0.21000000000000002 0.01 0.5
- link link_35: geometry collision box size=0.01 0.21000000000000002 0.5; visual box size=0.01 0.21000000000000002 0.5
- link link_36: geometry collision box size=0.21000000000000002 0.01 0.5; visual box size=0.21000000000000002 0.01 0.5
- link link_37: geometry collision box size=0.01 0.21000000000000002 0.5; visual box size=0.01 0.21000000000000002 0.5
- link link_38: geometry collision box size=0.01 0.21000000000000002 0.5; visual box size=0.01 0.21000000000000002 0.5
- link link_39: geometry collision box size=0.21000000000000002 0.01 0.5; visual box size=0.21000000000000002 0.01 0.5
- link link_4: geometry collision box size=0.21000000000000002 0.01 0.5; visual box size=0.21000000000000002 0.01 0.5
- link link_40: geometry collision box size=0.01 0.21000000000000002 0.5; visual box size=0.01 0.21000000000000002 0.5
- link link_41: geometry collision box size=0.21000000000000002 0.01 0.5; visual box size=0.21000000000000002 0.01 0.5
- link link_42: geometry collision box size=0.01 0.21000000000000002 0.5; visual box size=0.01 0.21000000000000002 0.5
- link link_43: geometry collision box size=0.21000000000000002 0.01 0.5; visual box size=0.21000000000000002 0.01 0.5
- link link_44: geometry collision box size=0.01 0.21000000000000002 0.5; visual box size=0.01 0.21000000000000002 0.5
- link link_45: geometry collision box size=0.21000000000000002 0.01 0.5; visual box size=0.21000000000000002 0.01 0.5
- link link_46: geometry collision box size=0.01 0.21000000000000002 0.5; visual box size=0.01 0.21000000000000002 0.5
- link link_47: geometry collision box size=0.21000000000000002 0.01 0.5; visual box size=0.21000000000000002 0.01 0.5
- link link_48: geometry collision box size=0.01 0.21000000000000002 0.5; visual box size=0.01 0.21000000000000002 0.5
- link link_49: geometry collision box size=0.21000000000000002 0.01 0.5; visual box size=0.21000000000000002 0.01 0.5
- link link_5: geometry collision box size=0.01 0.21000000000000002 0.5; visual box size=0.01 0.21000000000000002 0.5
- link link_50: geometry collision box size=0.01 0.21000000000000002 0.5; visual box size=0.01 0.21000000000000002 0.5
- link link_51: geometry collision box size=0.01 0.21000000000000002 0.5; visual box size=0.01 0.21000000000000002 0.5
- link link_52: geometry collision box size=0.21000000000000002 0.01 0.5; visual box size=0.21000000000000002 0.01 0.5
- link link_53: geometry collision box size=0.01 0.21000000000000002 0.5; visual box size=0.01 0.21000000000000002 0.5
- link link_54: geometry collision box size=0.21000000000000002 0.01 0.5; visual box size=0.21000000000000002 0.01 0.5
- link link_55: geometry collision box size=0.01 0.21000000000000002 0.5; visual box size=0.01 0.21000000000000002 0.5
- link link_56: geometry collision box size=0.21000000000000002 0.01 0.5; visual box size=0.21000000000000002 0.01 0.5
- link link_57: geometry collision box size=0.01 0.21000000000000002 0.5; visual box size=0.01 0.21000000000000002 0.5
- link link_58: geometry collision box size=0.21000000000000002 0.01 0.5; visual box size=0.21000000000000002 0.01 0.5
- link link_59: geometry collision box size=0.01 0.21000000000000002 0.5; visual box size=0.01 0.21000000000000002 0.5
- link link_6: geometry collision box size=0.21000000000000002 0.01 0.5; visual box size=0.21000000000000002 0.01 0.5
- link link_60: geometry collision box size=0.21000000000000002 0.01 0.5; visual box size=0.21000000000000002 0.01 0.5
- link link_61: geometry collision box size=0.01 0.21000000000000002 0.5; visual box size=0.01 0.21000000000000002 0.5
- link link_62: geometry collision box size=0.21000000000000002 0.01 0.5; visual box size=0.21000000000000002 0.01 0.5
- link link_63: geometry collision box size=0.01 0.21000000000000002 0.5; visual box size=0.01 0.21000000000000002 0.5
- link link_64: geometry collision box size=0.01 0.21000000000000002 0.5; visual box size=0.01 0.21000000000000002 0.5
- link link_65: geometry collision box size=0.21000000000000002 0.01 0.5; visual box size=0.21000000000000002 0.01 0.5
- link link_66: geometry collision box size=0.01 0.21000000000000002 0.5; visual box size=0.01 0.21000000000000002 0.5
- link link_67: geometry collision box size=0.21000000000000002 0.01 0.5; visual box size=0.21000000000000002 0.01 0.5
- link link_68: geometry collision box size=0.01 0.21000000000000002 0.5; visual box size=0.01 0.21000000000000002 0.5
- link link_69: geometry collision box size=0.21000000000000002 0.01 0.5; visual box size=0.21000000000000002 0.01 0.5
- link link_7: geometry collision box size=0.01 0.21000000000000002 0.5; visual box size=0.01 0.21000000000000002 0.5
- link link_70: geometry collision box size=0.01 0.21000000000000002 0.5; visual box size=0.01 0.21000000000000002 0.5
- link link_71: geometry collision box size=0.21000000000000002 0.01 0.5; visual box size=0.21000000000000002 0.01 0.5
- link link_72: geometry collision box size=0.01 0.21000000000000002 0.5; visual box size=0.01 0.21000000000000002 0.5
- link link_73: geometry collision box size=0.21000000000000002 0.01 0.5; visual box size=0.21000000000000002 0.01 0.5
- link link_74: geometry collision box size=0.01 0.21000000000000002 0.5; visual box size=0.01 0.21000000000000002 0.5
- link link_75: geometry collision box size=0.21000000000000002 0.01 0.5; visual box size=0.21000000000000002 0.01 0.5
- link link_76: geometry collision box size=0.01 0.21000000000000002 0.5; visual box size=0.01 0.21000000000000002 0.5
- link link_77: geometry collision box size=0.01 0.21000000000000002 0.5; visual box size=0.01 0.21000000000000002 0.5
- link link_78: geometry collision box size=0.21000000000000002 0.01 0.5; visual box size=0.21000000000000002 0.01 0.5
- link link_79: geometry collision box size=0.01 0.21000000000000002 0.5; visual box size=0.01 0.21000000000000002 0.5
- link link_8: geometry collision box size=0.21000000000000002 0.01 0.5; visual box size=0.21000000000000002 0.01 0.5
- link link_80: geometry collision box size=0.21000000000000002 0.01 0.5; visual box size=0.21000000000000002 0.01 0.5
- link link_81: geometry collision box size=0.01 0.21000000000000002 0.5; visual box size=0.01 0.21000000000000002 0.5
- link link_82: geometry collision box size=0.21000000000000002 0.01 0.5; visual box size=0.21000000000000002 0.01 0.5
- link link_83: geometry collision box size=0.01 0.21000000000000002 0.5; visual box size=0.01 0.21000000000000002 0.5
- link link_84: geometry collision box size=0.21000000000000002 0.01 0.5; visual box size=0.21000000000000002 0.01 0.5
- link link_85: geometry collision box size=0.01 0.21000000000000002 0.5; visual box size=0.01 0.21000000000000002 0.5
- link link_86: geometry collision box size=0.21000000000000002 0.01 0.5; visual box size=0.21000000000000002 0.01 0.5
- link link_87: geometry collision box size=0.01 0.21000000000000002 0.5; visual box size=0.01 0.21000000000000002 0.5
- link link_88: geometry collision box size=0.21000000000000002 0.01 0.5; visual box size=0.21000000000000002 0.01 0.5
- link link_89: geometry collision box size=0.01 0.21000000000000002 0.5; visual box size=0.01 0.21000000000000002 0.5
- link link_9: geometry collision box size=0.01 0.21000000000000002 0.5; visual box size=0.01 0.21000000000000002 0.5
- link link_90: geometry collision box size=0.01 0.21000000000000002 0.5; visual box size=0.01 0.21000000000000002 0.5
- link link_91: geometry collision box size=0.21000000000000002 0.01 0.5; visual box size=0.21000000000000002 0.01 0.5
- link link_92: geometry collision box size=0.01 0.21000000000000002 0.5; visual box size=0.01 0.21000000000000002 0.5
- link link_93: geometry collision box size=0.21000000000000002 0.01 0.5; visual box size=0.21000000000000002 0.01 0.5
- link link_94: geometry collision box size=0.01 0.21000000000000002 0.5; visual box size=0.01 0.21000000000000002 0.5
- link link_95: geometry collision box size=0.21000000000000002 0.01 0.5; visual box size=0.21000000000000002 0.01 0.5
- link link_96: geometry collision box size=0.01 0.21000000000000002 0.5; visual box size=0.01 0.21000000000000002 0.5
- link link_97: geometry collision box size=0.21000000000000002 0.01 0.5; visual box size=0.21000000000000002 0.01 0.5
- link link_98: geometry collision box size=0.01 0.21000000000000002 0.5; visual box size=0.01 0.21000000000000002 0.5
- link link_99: geometry collision box size=0.21000000000000002 0.01 0.5; visual box size=0.21000000000000002 0.01 0.5
Joints:
- removed joint joint_123
- removed joint joint_124
- removed joint joint_125
- removed joint joint_126
- removed joint joint_127
- removed joint joint_128
- removed joint joint_129
- removed joint joint_130
- removed joint joint_131
- removed joint joint_132
- removed joint joint_133
- removed joint joint_134
- removed joint joint_135
- removed joint joint_136
- removed joint joint_137
- removed joint joint_138
- removed joint joint_139
- removed joint joint_140
- removed joint joint_141
- removed joint joint_142
- removed joint joint_143
- removed joint joint_144
- removed joint joint_145
- removed joint joint_146
- removed joint joint_147
- removed joint joint_148
- removed joint joint_149
- removed joint joint_150
- removed joint joint_151
- removed joint joint_152
- removed joint joint_153
- removed joint joint_154
- removed joint joint_155
- removed joint joint_156
- removed joint joint_157
- removed joint joint_158
- removed joint joint_159
- removed joint joint_160
- removed joint joint_161
- removed joint joint_162
- removed joint joint_163
- removed joint joint_164
- removed joint joint_165
- removed joint joint_166
- removed joint joint_167
- removed joint joint_168
- removed joint joint_169
- removed joint joint_170
- removed joint joint_171
- removed joint joint_172
- removed joint joint_173
- removed joint joint_174
- removed joint joint_175
- removed joint joint_176
- removed joint joint_177
- removed joint joint_178
- removed joint joint_179
- removed joint joint_180
- removed joint joint_181
- removed joint joint_182
- removed joint joint_183
- removed joint joint_184
- removed joint joint_185
- removed joint joint_186
- removed joint joint_187
- removed joint joint_188
- removed joint joint_189
- removed joint joint_190
- removed joint joint_191
- removed joint joint_192
- removed joint joint_193
- removed joint joint_194
- removed joint joint_195
- removed joint joint_196
- removed joint joint_197
- removed joint joint_198
- removed joint joint_199
- removed joint joint_200
- removed joint joint_201
- removed joint joint_202
- removed joint joint_203
- removed joint joint_204
- removed joint joint_205
- removed joint joint_206
- removed joint joint_207
- removed joint joint_208
- removed joint joint_209
- removed joint joint_210
- removed joint joint_211
- removed joint joint_212
- removed joint joint_213
- removed joint joint_214
- removed joint joint_215
- removed joint joint_216
- removed joint joint_217
- removed joint joint_218
- removed joint joint_219
- removed joint joint_220
- removed joint joint_221
- removed joint joint_222
- removed joint joint_223
- removed joint joint_224
- removed joint joint_225
- removed joint joint_226
- removed joint joint_227
- removed joint joint_228
- removed joint joint_229
- removed joint joint_230
- removed joint joint_231
- removed joint joint_232
- removed joint joint_233
- removed joint joint_234
- removed joint joint_235
- removed joint joint_236
- removed joint joint_237
- removed joint joint_238
- removed joint joint_239
- removed joint joint_240
- removed joint joint_241
- removed joint joint_242
- removed joint joint_243
- removed joint joint_244
- removed joint joint_245
- removed joint joint_246
- removed joint joint_247
- removed joint joint_248
- removed joint joint_249
- removed joint joint_250
- removed joint joint_251
- removed joint joint_252
- removed joint joint_253
- removed joint joint_254
- removed joint joint_255
- removed joint joint_256
- removed joint joint_257
- removed joint joint_258
- removed joint joint_259
- removed joint joint_260
- removed joint joint_261
