Commit message: Arg parsing and implemented 2-person 2-shelf experiment

File: urdfs/generated/maze.urdf (robot description, URDF)
Before this commit: robot maze, 149 links, 148 joints
Links:
- removed link link_146
- removed link link_147
- link link_107: geometry collision box size=0.01 0.11 0.5; visual box size=0.01 0.11 0.5
- link link_11: geometry collision box size=0.11 0.01 0.5; visual box size=0.11 0.01 0.5
- link link_111: geometry collision box size=0.11 0.01 0.5; visual box size=0.11 0.01 0.5
- link link_112: geometry collision box size=0.11 0.01 0.5; visual box size=0.11 0.01 0.5
- link link_114: geometry collision box size=0.11 0.01 0.5; visual box size=0.11 0.01 0.5
- link link_116: geometry collision box size=0.01 0.11 0.5; visual box size=0.01 0.11 0.5
- link link_122: geometry collision box size=0.01 0.11 0.5; visual box size=0.01 0.11 0.5
- link link_123: geometry collision box size=0.01 0.11 0.5; visual box size=0.01 0.11 0.5
- link link_128: geometry collision box size=0.11 0.01 0.5; visual box size=0.11 0.01 0.5
- link link_129: geometry collision box size=0.11 0.01 0.5; visual box size=0.11 0.01 0.5
- link link_15: geometry collision box size=0.01 0.11 0.5; visual box size=0.01 0.11 0.5
- link link_20: geometry collision box size=0.01 0.11 0.5; visual box size=0.01 0.11 0.5
- link link_21: geometry collision box size=0.11 0.01 0.5; visual box size=0.11 0.01 0.5
- link link_25: geometry collision box size=0.01 0.2 0.25; visual box size=0.01 0.2 0.25
- link link_27: geometry collision box size=0.01 0.2 0.25; visual box size=0.01 0.2 0.25
- link link_29: geometry collision box size=0.01 0.11 0.5; visual box size=0.01 0.11 0.5
- link link_31: geometry collision box size=0.11 0.01 0.5; visual box size=0.11 0.01 0.5
- link link_36: geometry collision box size=0.01 0.11 0.5; visual box size=0.01 0.11 0.5
- link link_39: geometry collision box size=0.2 0.01 0.25; visual box size=0.2 0.01 0.25
- link link_43: geometry collision box size=0.01 0.2 0.25; visual box size=0.01 0.2 0.25
- link link_44: geometry collision box size=0.01 0.11 0.5; visual box size=0.01 0.11 0.5
- link link_47: geometry collision box size=0.11 0.01 0.5; visual box size=0.11 0.01 0.5
- link link_49: geometry collision box size=0.11 0.01 0.5; visual box size=0.11 0.01 0.5
- link link_53: geometry collision box size=0.01 0.11 0.5; visual box size=0.01 0.11 0.5
- link link_55: geometry collision box size=0.11 0.01 0.5; visual box size=0.11 0.01 0.5
- link link_56: geometry collision box size=0.01 0.11 0.5; visual box size=0.01 0.11 0.5
- link link_57: geometry collision box size=0.11 0.01 0.5; visual box size=0.11 0.01 0.5
- link link_58: geometry collision box size=0.11 0.01 0.5; visual box size=0.11 0.01 0.5
- link link_6: geometry collision box size=0.11 0.01 0.5; visual box size=0.11 0.01 0.5
- link link_60: geometry collision box size=0.11 0.01 0.5; visual box size=0.11 0.01 0.5
- link link_61: geometry collision box size=0.11 0.01 0.5; visual box size=0.11 0.01 0.5
- link link_62: geometry collision box size=0.11 0.01 0.5; visual box size=0.11 0.01 0.5
- link link_63: geometry collision box size=0.01 0.11 0.5; visual box size=0.01 0.11 0.5
- link link_67: geometry collision box size=0.01 0.11 0.5; visual box size=0.01 0.11 0.5
- link link_69: geometry collision box size=0.01 0.11 0.5; visual box size=0.01 0.11 0.5
- link link_70: geometry collision box size=0.01 0.11 0.5; visual box size=0.01 0.11 0.5
- link link_71: geometry collision box size=0.01 0.11 0.5; visual box size=0.01 0.11 0.5
- link link_73: geometry collision box size=0.2 0.01 0.25; visual box size=0.2 0.01 0.25
- link link_74: geometry collision box size=0.01 0.11 0.5; visual box size=0.01 0.11 0.5
- link link_75: geometry collision box size=0.11 0.01 0.5; visual box size=0.11 0.01 0.5
- link link_76: geometry collision box size=0.01 0.11 0.5; visual box size=0.01 0.11 0.5
- link link_77: geometry collision box size=0.11 0.01 0.5; visual box size=0.11 0.01 0.5
- link link_78: geometry collision box size=0.11 0.01 0.5; visual box size=0.11 0.01 0.5
- link link_79: geometry collision box size=0.11 0.01 0.5; visual box size=0.11 0.01 0.5
- link link_8: geometry collision box size=0.01 0.11 0.5; visual box size=0.01 0.11 0.5
- link link_80: geometry collision box size=0.01 0.11 0.5; visual box size=0.01 0.11 0.5
- link link_81: geometry collision box size=0.01 0.11 0.5; visual box size=0.01 0.11 0.5
- link link_90: geometry collision box size=0.2 0.01 0.25; visual box size=0.2 0.01 0.25
- link link_91: geometry collision box size=0.11 0.01 0.5; visual box size=0.11 0.01 0.5
- link link_94: geometry collision box size=0.11 0.01 0.5; visual box size=0.11 0.01 0.5
- link link_95: geometry collision box size=0.01 0.11 0.5; visual box size=0.01 0.11 0.5
- link link_96: geometry collision box size=0.11 0.01 0.5; visual box size=0.11 0.01 0.5
- link link_97: geometry collision box size=0.11 0.01 0.5; visual box size=0.11 0.01 0.5
- link link_99: geometry collision box size=0.01 0.11 0.5; visual box size=0.01 0.11 0.5
Joints:
- removed joint joint_146
- removed joint joint_147
